File: ESC_2Layer.sch (KiCad schematic (older format))
At the start: 79 parts, among them J1 SWD, Q1 PSMN011-30YLC, Q2 PSMN011-30YLC, Q3 PSMN011-30YLC, Q4 PSMN011-30YLC, Q5 PSMN011-30YLC, Q6 PSMN011-30YLC, U1 MIC4604, U2 MIC4604, U3 MIC4604, U4 STM32F030K6Tx, U5 AP1117-33

Commit message: Added PWM input
Connections:
- net labels added: DBG_PIN, PWM_IN, UART1_RX, UART1_TX
- wire segments 363 -> 367
- no-connect marks 14 -> 10
Changed lines of the file:
@@
 NoConn ~ 10475 2250
 NoConn ~ 10475 2350
-NoConn ~ 10475 2450
 NoConn ~ 10475 2550
 NoConn ~ 10475 2950
@@
 NoConn ~ 6275 2550
 NoConn ~ 6275 3050
-NoConn ~ 6275 3150
-NoConn ~ 6275 3250
-NoConn ~ 6275 3350
 $Comp
 L device:R_Small R17
@@
 Wire Wire Line
 	925  7250 1525 7250
+Wire Wire Line
+	10475 2450 10825 2450
+Text Label 10825 2450 2    50   ~ 0
+PWM_IN
+Wire Wire Line
+	6275 3250 5825 3250
+Wire Wire Line
+	6275 3350 5825 3350
+Text Label 5825 3250 0    50   ~ 0
+UART1_TX
+Text Label 5825 3350 0    50   ~ 0
+UART1_RX
+Wire Wire Line
+	6275 3150 5825 3150
+Text Label 5825 3150 0    50   ~ 0
+DBG_PIN
 $EndSCHEMATC
